File: Battery-charging-cascade/bq24616_battery_charger.brd (EAGLE design)
At the start: 160 x 100 mm, 80 parts, among them J1 PJ-063BH, J2 S2B-PH, J3 DG301-2P", J4 DG301-2P", U1 BQ24616_RGE_24

Commit message: final routing for rewive
Parts:
- removed ACS, CEN, IS2, PG, ST1, ST2, VCC: TEST_PAD-[1.27MM], testing:TP1.27MM
- removed PAD1, PAD2, PAD3, PAD4: (no value), commonly used connectors:2,54/1,1
- added C20: 100nF, Capacitors:C0603
- added C21: 22pF, Capacitors:C0603
- added GND', SYS: TEST_RING, testing:TEST_RING
- added J5: S4B-PH-K, con-jst-ph:S4B-PH-K
- added SB2: SHORT, testing:SHORT
- C1, C2, C3, C4: value 10 uF -> 10uF
- C5: value 2.2 uF -> 2.2uF, 50V
- GND, OUT: value TEST_PAD-[1.27MM] -> TEST_RING; device testing:TP1.27MM -> testing:TEST_RING
- moved J4 134.7 mm to (56.4, 29.0), turned to 90 degrees
- moved J3 127.2 mm to (56.4, 11.5), turned to 90 degrees
- moved R21 118.0 mm to (41.8, 5.61), turned to 270 degrees
- moved R20 111.6 mm to (39.6, 5.61), turned to 270 degrees
- moved Q3 111.2 mm to (51.5, 20.0), turned to 270 degrees
- moved C3 108.7 mm to (49.5, 10.5), turned to 270 degrees
- moved PAD6 108.3 mm to (5.95, 31.5)
- moved C12 107.9 mm to (43.0, 15.5), turned to 270 degrees
- moved R19 105.5 mm to (37.4, 5.61), turned to 270 degrees
- moved OUT 103.7 mm to (56.4, 18.7)
- moved R15 103.7 mm to (33.0, 5.61), turned to 90 degrees
- moved GND 103.0 mm to (52.5, 3.00)
- moved CTT 101.9 mm to (31.5, 13.1)
- moved C11 100.8 mm to (42.9, 18.8), turned to 180 degrees
- moved C2 100.7 mm to (49.8, 28.4), turned to 90 degrees
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Connections:
- net N$10 renamed REGN
- net N$11 renamed PH
- net N$12 renamed BTST1
- net N$13 renamed BTST
- net N$15 renamed BATDRV
- net N$18 renamed TCC
- net N$2 renamed VCC1
- net N$20 renamed TS
- net N$4 renamed GATE
- net N$5 renamed LODRV
- net N$7 renamed ACDRV
- net N$8 renamed HIDRV
- net N$9 renamed ACP
- removed net N$14: R8.2, R9.1, U1.12, VFB.1
- removed net N$16: C13.1, R10.2, U1.24, VCC.1
- new net VCC: C13.1, R10.2, U1.24
- new net VFB: C21.2, R8.2, R9.1, U1.12, VFB.1
- net ACSET: no longer ACS.1
- net AGND: now also GND'.1, J4.2, SB2.2; no longer C10.2, CTTC.2, J4.1, PAD2.1, PAD4.1, U1.17, U1.25, U1.V, U1.V_1, U1.V_2, U1.V_3, U1.V_4, U1.V_5, U1.V_6, U1.V_7, U1.V_8
- net CHARGE_EN: now also J5.1; no longer CEN.1
- net GND: now also C10.2, C20.2, CTTC.2, SB2.1, U1.17, U1.25, U1.V, U1.V_1, U1.V_2, U1.V_3, U1.V_4, U1.V_5, U1.V_6, U1.V_7, U1.V_8
- net ISET2: no longer IS2.1
- net POWER_GOOD: now also J5.2; no longer PG.1
- net SRN: now also C20.1, C21.1; no longer PAD1.1
- net STAT1: now also J5.4; no longer ST1.1
- net STAT2: now also J5.3; no longer ST2.1
- net SYSTEM+: now also J4.1, SYS.1; no longer J4.2, PAD3.1
Routing:
- net VREF: track 0.00 -> 36.2 mm
- net CHARGE_EN: track 0.00 -> 34.7 mm, vias 0 -> 1
- net POWER_GOOD: track 0.00 -> 23.7 mm, vias 0 -> 1
- net STAT2: track 0.00 -> 22.7 mm, vias 0 -> 1
- net GATE: track 0.00 -> 22.4 mm
- net ACDRV: track 0.00 -> 19.2 mm
- net LODRV: track 0.00 -> 19.1 mm, vias 0 -> 2
- net BATDRV: track 0.00 -> 18.9 mm, vias 0 -> 2
- net STAT1: track 0.00 -> 18.7 mm
- net ACSET: track 0.00 -> 18.4 mm, vias 0 -> 2
- net ISET2: track 0.00 -> 15.9 mm, vias 0 -> 2
- net VFB: track 0.00 -> 14.7 mm
- net ACP: track 0.00 -> 14.1 mm, vias 0 -> 5
- net SRN: track 0.00 -> 12.8 mm, vias 0 -> 9
- net N$22: track 0.00 -> 12.6 mm
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- added copper zone on layer 1, net ACP
- added copper zone on layer 16, net ACP
- added copper zone on layer 1, net ADAPTER+
- added copper zone on layer 16, net ADAPTER+
- added copper zone on layer 1, net AGND
- added copper zone on layer 16, net AGND
- added copper zone on layer 1, net GND
- added copper zone on layer 16, net GND
- added copper zone on layer 1, net N$17
- added copper zone on layer 1, net N$3
- added copper zone on layer 1, net PH
- added copper zone on layer 16, net PH
- added copper zone on layer 1, net SRN
- added copper zone on layer 16, net SRN
- added copper zone on layer 1, net SRP
- added copper zone on layer 1, net SYSTEM+
- added copper zone on layer 16, net SYSTEM+
- added copper zone on layer 1, net VCC1
- added copper zone on layer 16, net VCC1
Other:
- board size 160 x 100 mm -> 60 x 40 mm

Commit message: ready to manufacturing
Parts:
- removed SB1: SOLDER_BRIDGE, testing:SOLDER_BRIDGE
- added CEN_VREF: SOLDER_BRIDGE, testing:SOLDER_BRIDGE
- J5: value S4B-PH-K -> S6B-PH-K; device con-jst-ph:S4B-PH-K -> con-jst-ph:S6B-PH-K
- moved C21 3.04 mm to (43.4, 12.7), turned to 180 degrees
- moved C20 1.90 mm to (39.6, 14.5), turned to 180 degrees
- moved R7 1.08 mm to (33.1, 21.7), turned to 90 degrees
- moved C12 0.63 mm to (43.7, 15.5)
- moved J3 0.63 mm to (55.8, 11.5)
- moved J4 0.63 mm to (55.8, 29.0)
- moved D1 0.53 mm to (37.3, 20.7)
- moved C9 0.53 mm to (37.3, 23.4), turned to 90 degrees
- moved OUT 0.51 mm to (55.9, 18.7)
- moved SYS 0.51 mm to (55.9, 22.0)
- moved R10 0.46 mm to (29.5, 21.3)
- moved R13 0.38 mm to (26.7, 10.2)
- moved J5 0.32 mm to (18.3, 5.58)
- moved R5 0.30 mm to (16.0, 23.3)
- moved C16 0.25 mm to (28.7, 10.2)
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- renumbered PAD5 to POWER, PAD6 to GROUND
Connections:
- net CHARGE_EN: now also CEN_VREF.1, J5.5; no longer J5.1, SB1.1
- net GND: now also J5.1
- net VREF: now also CEN_VREF.2, J5.6; no longer SB1.2
Routing:
- net GND: track 5.56 -> 28.9 mm, vias 11 -> 13
- net CHARGE_EN: track 34.7 -> 23.7 mm
- net STAT2: track 22.7 -> 25.8 mm
- net ACP: track 14.1 -> 11.1 mm
- net POWER_GOOD: track 23.7 -> 26.2 mm
- net PH: track 6.90 -> 8.96 mm
- net HIDRV: track 11.5 -> 13.2 mm
- net BTST1: track 4.26 -> 5.48 mm, vias 0 -> 2
- net STAT1: track 18.7 -> 17.6 mm
- net SRN: track 12.8 -> 12.0 mm, vias 9 -> 12
- net REGN: track 5.33 -> 4.63 mm
- added copper zone on layer 1, net VCC
Other:
- board text added: "10k ntc"
- board text added: "ACS"
- board text added: "C:/Users/User/Desktop/123.bmp"
- board text added: "CEN"
- board text added: "GND"
- board text added: "IS2"
- board text added: "PG"
- board text added: "ST1"
- board text added: "ST2"
- board text added: "VREF"
