File: Battery-charging-cascade/bq24616_battery_charger.sch (EAGLE design)
At the start: 57 parts, among them J1 PJ-063BH, J2 S2B-PH-K, U1 BQ24616_RGE_24

Commit message: schematic for review
Parts:
- added ACDR, ACS, CEN, CTT, GND, IS1, IS2, PG, ST1, ST2, VFB: TEST_PAD-[1.27MM], testing:TEST_PAD-[1.27MM]
- added C17, C18, C19: 100nF, Capacitors:C-EU-CERAMIC0603
- added J3, J4: DG301-2P", Terminal blocks:DG301-2P"
- added PAD1, PAD2, PAD3, PAD4, PAD5, PAD6: (no value), commonly used connectors:WIRE_TO_BOARD_2,54/1,1
- added SB1: SOLDER_BRIDGE, testing:SOLDER_BRIDGE
- C10: value 1uF -> 1uF, 16V
- C9: value 100nF -> 100nF, 50V
- CTTC: value (none) -> 33nF
- D2: value LED0805 -> ST1_Blue
- D3: value LED0805 -> ST2_Blue
- D4: value LED0805 -> PG_Green
- J2: value S2B-PH-K -> S2B-PH
- R11: value (none) -> 1k
- R13: value (none) -> 100
- R14: value (none) -> 1.78k
- R15: value (none) -> 4.99k
- R16, R17: value (none) -> 10k
- R18, R22: value (none) -> 3k3
- R19, R20: value (none) -> 51k
- R21, R9: value (none) -> 102k
- R23: value (none) -> 1k6
- R24: value (none) -> 13k7
- R8: value (none) -> 510k
Connections:
- removed net N$6: C1.1, C14.1, C2.1, C6.2, Q3.S, Q4.D, R1.2, R12.1, U1.ACN
- new net SYSTEM+: C1.1, C14.1, C2.1, C6.2, J4.2, PAD3.P, Q3.S, Q4.D, R1.2, R12.1, U1.ACN
- net ACSET: now also ACS.P$1, C17.1, R21.1, R24.2
- net ADAPTER+: now also PAD5.P
- net AGND: now also C1.2, C10.2, C2.2, C3.2, C4.2, GND.P$1, J3.1, J4.1, PAD2.P, PAD4.P, PAD6.P; no longer C11.2, C13.2, C15.2, C16.2, C7.2, R15.2, R9.2
- net CHARGE_EN: now also CEN.P$1, SB1.1
- net GND: now also C11.2, C13.2, C15.2, C16.2, C17.2, C18.2, C19.2, C7.2, J2.2, R15.2, R22.1, R23.1, R24.1, R9.2; no longer C1.2, C10.2, C2.2, C3.2, C4.2
- net ISET1: now also C18.1, IS1.P$1, R19.1, R22.2
- net ISET2: now also C19.1, IS2.P$1, R20.1, R23.2
- net N$14: now also VFB.P$1
- net N$18: now also CTT.P$1
- net N$22: now also J2.1
- net N$4: now also ACDR.P$1
- net POWER_GOOD: now also PG.P$1
- net SRN: now also J3.2, PAD1.P
- net STAT1: now also ST1.P$1
- net STAT2: now also ST2.P$1
- net VREF: now also R19.2, R20.2, R21.2, SB1.2
Other:
- note added: "50V"
- note added: "AGND means Adapter Ground: Hight voltage power path ground GND is low voltage ground of internal IC circiutry"
- note added: "CTTC cap. sets the fast charge safety timer. 33nf is 3h timer"
- note added: "Hight side MOSFET driven by 15 + 6V = 21V (6V over input voltage)"
- note added: "NOTE that current limiting resistor R7 used in ref. design but not used in datasheet"
- note added: "R14, R15 voltage divider is specifically tuned for 10k Njiang Chinese ntc thermistor in stock"
- note added: "These nominals selected for testing purposes and sets 3A max adapter current 1A fast charging current 0.1A precharge current"
- note removed: "!!!"
- note removed: "AGND means Adapter Ground noizy analog ground"
- note removed: "CTTC cap. sets the fast charge safety timer"
- note removed: "Hight side MOSFET driven by INPUT+6V of GS Voltage"
- note removed: "PACK+"
- note removed: "PACK-"
- note removed: "R7 used in ref. design but not used in datasheet You need to check Bootstrap cap value according to FET Qgs"
- note removed: "SYSTEM+"
- note removed: "Testpoints!!!"
- moved on the sheet: C10, C13, C16, C9, D1, D2, D3, D4, R10, R13, R14, R15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

Commit message: final routing for rewive
Parts:
- removed ACS, CEN, IS2, PG, ST1, ST2, VCC: TEST_PAD-[1.27MM], testing:TEST_PAD-[1.27MM]
- removed PAD1, PAD2, PAD3, PAD4: (no value), commonly used connectors:WIRE_TO_BOARD_2,54/1,1
- added C20: 100nF, Capacitors:C-EU-CERAMIC0603
- added C21: 22pF, Capacitors:C-EU-CERAMIC0603
- added GND', SYS: TEST_RING, testing:TEST_RING
- added J5: S4B-PH-K, con-jst-ph:S4B-PH-K
- added SB2: SHORT, testing:SHORT
- C1, C2, C3, C4: value 10 uF -> 10uF
- C5: value 2.2 uF -> 2.2uF, 50V
- GND, OUT: value TEST_PAD-[1.27MM] -> TEST_RING; device testing:TEST_PAD-[1.27MM] -> testing:TEST_RING
Connections:
- net N$10 renamed REGN
- net N$11 renamed PH
- net N$12 renamed BTST1
- net N$13 renamed BTST
- net N$15 renamed BATDRV
- net N$18 renamed TCC
- net N$2 renamed VCC1
- net N$20 renamed TS
- net N$4 renamed GATE
- net N$5 renamed LODRV
- net N$7 renamed ACDRV
- net N$8 renamed HIDRV
- net N$9 renamed ACP
- removed net N$14: R8.2, R9.1, U1.VFB, VFB.P$1
- removed net N$16: C13.1, R10.2, U1.VCC, VCC.P$1
- new net VCC: C13.1, R10.2, U1.VCC
- new net VFB: C21.2, R8.2, R9.1, U1.VFB, VFB.P$1
- net ACSET: no longer ACS.P$1
- net AGND: now also GND'.P$1, J4.2, SB2.2; no longer C10.2, CTTC.2, J4.1, PAD2.P, PAD4.P, U1.EPAD, U1.GND
- net CHARGE_EN: now also J5.1; no longer CEN.P$1
- net GND: now also C10.2, C20.2, CTTC.2, SB2.1, U1.EPAD, U1.GND
- net ISET2: no longer IS2.P$1
- net POWER_GOOD: now also J5.2; no longer PG.P$1
- net SRN: now also C20.1, C21.1; no longer PAD1.P
- net STAT1: now also J5.4; no longer ST1.P$1
- net STAT2: now also J5.3; no longer ST2.P$1
- net SYSTEM+: now also J4.1, SYS.P$1; no longer J4.2, PAD3.P
Other:
- moved on the sheet: C1, D2, D3, D4, J3, J4, R16, R17, R18, VFB

Commit message: ready to manufacturing
Parts:
- removed SB1: SOLDER_BRIDGE, testing:SOLDER_BRIDGE
- added CEN_VREF: SOLDER_BRIDGE, testing:SOLDER_BRIDGE
- J5: value S4B-PH-K -> S6B-PH-K; device con-jst-ph:S4B-PH-K -> con-jst-ph:S6B-PH-K
- renumbered PAD5 to POWER, PAD6 to GROUND
Connections:
- net CHARGE_EN: now also CEN_VREF.1, J5.5; no longer J5.1, SB1.1
- net GND: now also J5.1
- net VREF: now also CEN_VREF.2, J5.6; no longer SB1.2
